File: PCB/Prototype.kicad_sch (KiCad schematic)
At the start: 7 parts, among them SW5 SW_Push, SW6 SW_Push, SW7 SW_Push, SW8 SW_Push, U1 XIAO-RP2040-DIP

Commit message: Initial commit!!
Parts:
- added SW1, SW2: SW_Push, Button_Switch_Keyboard:SW_Cherry_MX_1.00u_PCB, symbol Switch:SW_Push
Connections:
- net GND: now also SW1.1, SW2.1
- net at U1.6 (GPIO7/SCL): now also SW1.2
- net at U1.7 (GPIO0/TX): now also SW2.2
Other:
- moved on the sheet: D1, D2

Commit message: Finished build
Parts:
- added SW3: RotaryEncoder_Switch, Rotary_Encoder:RotaryEncoder_Alps_EC11E-Switch_Vertical_H20mm, symbol Device:RotaryEncoder_Switch
Connections:
- net GND: now also SW3.C, SW3.S1
- net at U1.1 (GPIO26/ADC0/A0): now also SW3.S2
- net at U1.2 (GPIO27/ADC1/A1): now also SW3.B
- net at U1.3 (GPIO28/ADC2/A2): now also SW3.A
